File: PCB/4ChannelAnalyzer/4ChannelAnalyzer.sch (EAGLE design)
At the start: 0 parts

Commit message: Added components to the PCB design
Parts:
- added LED1, LED2, LED3, LED4, LED5, LED6: LG_T679-E1F1-1, led:LG_T679-E1F1-1
- added LPC1: (no value), LPCXpresso_LPC1769:LPCXPRESSO_LPC1769
- added R1, R2, R3, R4, R5, R6: (no value), rcl:R-EU_M2012
- added U1, U2: ADS1015IDGST, ADS1015:ADS1015IDGST
- added X1, X2: (no value), con-wago255:233-108
- added X3: MINI-USB-32005-301, con-cypressindustries:MINI-USB-32005-301
