File: PCB/4ChannelAnalyzer/4ChannelAnalyzer.brd (EAGLE design)
At the start: 91.4 x 64.8 mm, 22 parts, among them U1-ADD-49 ADS1015IDGST, U2-ADD-48 ADS1015IDGST, U3 LM1117MP-3.3, X3 MINI-USB-32005-301

Commit message: Repositioning one of the PullUp resistors for I2C
Parts:
- moved R7 2.29 mm to (47.6, 24.1), turned to 180 degrees
Routing:
- net VCC3.3V: track 119.6 -> 118.6 mm
Changed lines of the file:
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@@
 <element name="C1" library="rcl" package="C0805" value="10uF" x="15.875" y="15.5575" rot="R270"/>
 <element name="C2" library="rcl" package="C0805" value="10uF" x="22.225" y="15.5575" rot="R180"/>
-<element name="R7" library="rcl" package="M0805" value="10K" x="46.355" y="26.035" rot="R270"/>
+<element name="R7" library="rcl" package="M0805" value="10K" x="47.625" y="24.13" rot="R180"/>
 <element name="R8" library="rcl" package="M0805" value="10K" x="56.515" y="21.9075"/>
 <element name="J1" library="con-amp" package="10X07MTA" value="" x="86.36" y="43.4975" rot="R90"/>
@@
 <wire x1="52.3494" y1="20.828" x2="50.927" y2="20.828" width="0.4064" layer="1"/>
 <wire x1="50.927" y1="20.828" x2="50.4825" y2="21.2725" width="0.4064" layer="1"/>
-<wire x1="50.4825" y1="21.2725" x2="50.4825" y2="28.575" width="0.4064" layer="1"/>
+<wire x1="50.4825" y1="21.2725" x2="50.4825" y2="24.13" width="0.4064" layer="1"/>
+<wire x1="50.4825" y1="24.13" x2="50.4825" y2="28.575" width="0.4064" layer="1"/>
 <wire x1="50.4825" y1="28.575" x2="49.8475" y2="29.21" width="0.4064" layer="1"/>
-<wire x1="49.8475" y1="29.21" x2="46.355" y2="29.21" width="0.4064" layer="1"/>
-<wire x1="46.355" y1="29.21" x2="29.21" y2="29.21" width="0.4064" layer="1"/>
+<wire x1="49.8475" y1="29.21" x2="29.21" y2="29.21" width="0.4064" layer="1"/>
 <wire x1="29.21" y1="29.21" x2="27.305" y2="31.115" width="0.4064" layer="1"/>
 <wire x1="27.305" y1="31.115" x2="27.305" y2="33.655" width="0.4064" layer="1"/>
 <contactref element="R7" pad="1"/>
-<wire x1="46.355" y1="26.985" x2="46.355" y2="29.21" width="0.8128" layer="1"/>
+<wire x1="48.575" y1="24.13" x2="50.4825" y2="24.13" width="0.8128" layer="1"/>
 </signal>
 <signal name="SCL48">
@@
 <wire x1="47.9806" y1="21.3106" x2="47.2694" y2="21.3106" width="0.4064" layer="1"/>
 <wire x1="47.2694" y1="21.3106" x2="46.6725" y2="21.9075" width="0.4064" layer="1"/>
+<wire x1="46.6725" y1="21.9075" x2="46.355" y2="21.9075" width="0" layer="19" extent="1-16"/>
 <wire x1="46.6725" y1="21.9075" x2="46.355" y2="21.9075" width="0.8128" layer="1"/>
-<wire x1="46.355" y1="21.9075" x2="44.1325" y2="21.9075" width="0.8128" layer="1"/>
 <contactref element="R7" pad="2"/>
 <contactref element="R8" pad="2"/>
+<wire x1="46.355" y1="21.9075" x2="44.1325" y2="21.9075" width="0.8128" layer="1"/>
 <wire x1="52.3494" y1="20.32" x2="57.4675" y2="20.32" width="0.4064" layer="1"/>
 <wire x1="57.4675" y1="20.32" x2="77.1144" y2="20.32" width="0.4064" layer="1"/>
-<wire x1="46.355" y1="25.085" x2="46.355" y2="21.9075" width="0.8128" layer="1"/>
 <wire x1="57.465" y1="21.9075" x2="57.465" y2="20.3225" width="0.8128" layer="1"/>
 <wire x1="57.465" y1="20.3225" x2="57.4675" y2="20.32" width="0.8128" layer="1"/>
+<wire x1="46.6725" y1="21.9075" x2="46.675" y2="21.9075" width="0.8128" layer="1"/>
+<wire x1="46.675" y1="21.9075" x2="46.675" y2="24.13" width="0.8128" layer="1"/>
 </signal>
 </signals>
